Commit message: description/ros2_control.xacro: Added bucket ladder lift and buckets joints

File: description/ros2_control.xacro (robot description, xacro)
@@ -37,4 +37,16 @@
             <state_interface name="velocity" />
         </joint>
+        <joint name="bucket_ladder_lift_joint">
+            <command_interface name="position">
+                <param name="min">-1</param>
+                <param name="max">1</param>
+            </command_interface>
+            <state_interface name="position" />
+        </joint>
+        <joint name="bucket_ladder_buckets_joint">
+            <command_interface name="velocity" />
+            <state_interface name="position" />
+            <state_interface name="velocity" />
+        </joint>
     </ros2_control>
   </xacro:macro>

Commit message: description/ros2_control.xacro: Added dump bucket joint

File: description/ros2_control.xacro (robot description, xacro)
@@ -49,4 +49,11 @@
             <state_interface name="velocity" />
         </joint>
+        <joint name="bucket_dump_joint">
+            <command_interface name="position">
+                <param name="min">-1</param>
+                <param name="max">1</param>
+            </command_interface>
+            <state_interface name="position" />
+        </joint>
     </ros2_control>
   </xacro:macro>

Commit message: description/ros2_control.xacro: Added bucket ladder frame joint

File: description/ros2_control.xacro (robot description, xacro)
@@ -36,4 +36,11 @@
             <state_interface name="position" />
             <state_interface name="velocity" />
+        </joint>
+        <joint name="bucket_ladder_frame_joint">
+            <command_interface name="position">
+                <param name="min">0</param>
+                <param name="max">1</param>
+            </command_interface>
+            <state_interface name="position" />
         </joint>
         <joint name="bucket_ladder_lift_joint">

Commit message: description/ros2_control.xacro: Modified to support 4 diff hardware plugins
- Modified to support robot, mock, ign_gazebo, and gazebo hardware and
  related plugin files

File: description/ros2_control.xacro (robot description, xacro)
@@ -1,7 +1,7 @@
 <?xml version="1.0"?>
 <robot xmlns:xacro="http://www.ros.org/wiki/xacro">
-  <xacro:macro name="ros2_control" params="use_mock_hardware">
+  <xacro:macro name="ros2_control" params="use_hardware">
     <ros2_control name="ros2_control" type="system">
-       <xacro:unless value="${use_mock_hardware}">
+       <xacro:if value="${use_hardware == 'robot'}">
             <hardware>
                 <plugin>robot_hardware_interface/RobotSystemHardware</plugin>
@@ -9,10 +9,19 @@
                 <param name="hw_stop_duration_sec">3.0</param>
             </hardware>
-        </xacro:unless>
-        <xacro:if value="${use_mock_hardware}">
+        </xacro:if>
+        <xacro:if value="${use_hardware == 'mock'}">
             <hardware>
-                <!-- <plugin>gazebo_ros2_control/GazeboSystem</plugin> -->
                 <plugin>mock_components/GenericSystem</plugin>
                 <param name="calculate_dynamics">true</param>
+            </hardware>
+        </xacro:if>
+        <xacro:if value="${use_hardware == 'ign_gazebo'}">
+            <hardware>
+                <plugin>gz_ros2_control/GazeboSimSystem</plugin>
+            </hardware>
+        </xacro:if>
+        <xacro:if value="${use_hardware == 'gazebo'}">
+            <hardware>
+                <plugin>gazebo_ros2_control/GazeboSystem</plugin>
             </hardware>
         </xacro:if>
@@ -117,11 +126,22 @@
         </gpio>
     </ros2_control>
+    <xacro:if value="${use_hardware == 'ign_gazebo'}">
+        <gazebo>
+            <plugin filename="libgz_ros2_control-system.so" name="gz_ros2_control::GazeboSimROS2ControlPlugin">
+                <robot_param>robot_description</robot_param>
+                <robot_param_node>robot_state_publisher</robot_param_node>
+                <parameters>$(find osprey_ros)/config/robot_controllers.yaml</parameters>
+            </plugin>
+        </gazebo>
+    </xacro:if>
+    <xacro:if value="${use_hardware == 'gazebo'}">
+        <gazebo>
+            <plugin filename="libgazebo_ros2_control.so" name="gazebo_ros2_control::GazeboSystemInterface">
+                <robot_param>robot_description</robot_param>
+                <robot_param_node>robot_state_publisher</robot_param_node>
+                <parameters>$(find osprey_ros)/config/robot_controllers.yaml</parameters>
+            </plugin>
+        </gazebo>
+    </xacro:if>
   </xacro:macro>
-    <gazebo>
-        <plugin filename="libgazebo_ros2_control.so" name="gazebo_ros2_control">
-            <robot_param>robot_description</robot_param>
-            <robot_param_node>robot_state_publisher</robot_param_node>
-            <parameters>$(find osprey_ros)/config/robot_controllers.yaml</parameters>
-        </plugin>
-    </gazebo>
 </robot>
