Commit message: description/inertial_macros.xacro: Modify cylinder inertial to be hollow

File: description/inertial_macros.xacro (robot description, xacro)
@@ -14,7 +14,7 @@
             <xacro:insert_block name="origin"/>
             <mass value="${mass}" />
-            <inertia ixx="${(1/12) * mass * (3*radius*radius + length*length)}" ixy="0.0" ixz="0.0"
-                    iyy="${(1/12) * mass * (3*radius*radius + length*length)}" iyz="0.0"
-                    izz="${(1/2) * mass * (radius*radius)}" />
+            <inertia ixx="${(1/12) * mass * (3*(radius*radius + 0.00064516) + length*length)}" ixy="0.0" ixz="0.0"
+                    iyy="${(1/12) * mass * (3*(radius*radius + 0.00064516) + length*length)}" iyz="0.0"
+                    izz="${(1/2) * mass * (radius*radius + 0.00064516)}" />
         </inertial>
     </xacro:macro>
