Commit message: description/robot.urdf.xacro: Conditionally include gazebo tags & plugins

File: description/robot.urdf.xacro (robot description, xacro)
@@ -6,4 +6,10 @@
 	<xacro:include filename="robot_core.xacro" />
 	<xacro:include filename="ros2_control.xacro" />
+    <xacro:macro name="gazebo" params="use_hardware">
+      <xacro:if value="${use_hardware == 'ign_gazebo'}">
+	    <xacro:include filename="gazebo_plugins.xacro" />
+      </xacro:if>
+    </xacro:macro>
+	<xacro:gazebo use_hardware="$(arg use_hardware)"/>
 	<xacro:ros2_control use_hardware="$(arg use_hardware)"/>
 </robot>

Commit message: description/robot.urdf.xacro: Added year variable to control which robot
- Default is empty, can be set to 24 for the 2024 robot, pending other
  changes to launch files, etc

File: description/robot.urdf.xacro (robot description, xacro)
@@ -1,9 +1,13 @@
 <?xml version="1.0"?>
 <robot xmlns:xacro="http://www.ros.org/wiki/xacro"  name="opsrey_ros">
+	<xacro:arg name="year" default="" />
 	<xacro:arg name="use_hardware" default="robot" />
 	<xacro:include filename="colors.xacro" />
 	<xacro:include filename="inertial_macros.xacro" />
-	<xacro:include filename="robot_core.xacro" />
-	<xacro:include filename="ros2_control.xacro" />
+    <xacro:macro name="robot_year" params="year">
+        <xacro:include filename="robot${year}_core.xacro" />
+        <xacro:include filename="robot${year}_ros2_control.xacro" />
+	    <xacro:ros2_control use_hardware="$(arg use_hardware)"/>
+    </xacro:macro>
     <xacro:macro name="gazebo" params="use_hardware">
       <xacro:if value="${use_hardware == 'ign_gazebo'}">
@@ -11,5 +15,5 @@
       </xacro:if>
     </xacro:macro>
+	<xacro:robot_year year="$(arg year)"/>
 	<xacro:gazebo use_hardware="$(arg use_hardware)"/>
-	<xacro:ros2_control use_hardware="$(arg use_hardware)"/>
 </robot>
