Commit message: description/robot_core.xacro: Fix axis aligment and center
- Move to a 0 based center of the robot, front is negative offset and
  rear is positive offset from 1/2 the length/width from center
- Correct measurement values

File: description/robot_core.xacro (robot description, xacro)
@@ -4,9 +4,12 @@
     <xacro:property name="limit_velocity" value="1" />
     <!-- Values in meters -->
-    <xacro:property name="chassis_length" value="0.762" />
+    <xacro:property name="chassis_length" value="0.8128" />
     <xacro:property name="chassis_height" value="0.0889" />
-    <xacro:property name="chassis_width" value="0.368" />
-    <xacro:property name="wheel_length" value="0.1" />
-    <xacro:property name="wheel_radius" value="0.15" />
+    <xacro:property name="chassis_width" value="0.3556" />
+    <xacro:property name="wheel_length" value="0.1016" />
+    <xacro:property name="wheel_radius" value="0.1524" />
+    <xacro:property name="wheel_offset_front" value="${-chassis_length/2 + 0.1778}" />
+    <xacro:property name="wheel_offset_rear" value="${chassis_length/2 - 0.2286}" />
+    <xacro:property name="wheel_offset_side" value="${wheel_length/2 + chassis_width/2 + 0.0127}" />
     <link name="base_link"></link>
     <!-- Main Body/Chassis -->
@@ -14,9 +17,7 @@
         <parent link="base_link"/>
         <child link="chassis"/>
-        <origin xyz="-0.1 0 0"/>
     </joint>
     <link name="chassis">
         <collision>
-            <origin xyz="0.0935 0 0.00" rpy="0 0 0"/>
             <geometry>
                 <box size="${chassis_length} ${chassis_width} ${chassis_height}"/>
@@ -24,5 +25,4 @@
         </collision>
         <visual>
-            <origin xyz="${chassis_length/2} 0 0.00" rpy="0 0 0"/>
             <geometry>
                 <box size="${chassis_length} ${chassis_width} ${chassis_height}"/>
@@ -31,5 +31,5 @@
         </visual>
         <xacro:inertial_box mass="0.5" x="${chassis_length}" y="${chassis_width}" z="${chassis_height}">
-            <origin xyz="${chassis_length/2} 0 0.04675" rpy="0 0 0"/>
+            <origin xyz="${chassis_length/2} 0 0" rpy="0 0 0"/>
         </xacro:inertial_box>
     </link>
@@ -38,5 +38,5 @@
         <parent link="base_link"/>
         <child link="front_left_wheel"/>
-        <origin xyz="-0.0585 0.0725 0" rpy="-${pi/2} 0 0"/>
+        <origin xyz="${wheel_offset_front} ${wheel_offset_side} 0" rpy="-${pi/2} 0 0"/>
         <axis xyz="0 0 1"/>
         <limit effort="${limit_effort}" velocity="${limit_velocity}"/>
@@ -62,5 +62,5 @@
         <parent link="base_link"/>
         <child link="front_right_wheel"/>
-        <origin xyz="-0.0585 -0.0725 0" rpy="${pi/2} 0 0"/>
+        <origin xyz="${wheel_offset_front} -${wheel_offset_side} 0" rpy="${pi/2} 0 0"/>
         <axis xyz="0 0 -1"/>
         <limit effort="${limit_effort}" velocity="${limit_velocity}"/>
@@ -86,5 +86,5 @@
         <parent link="base_link"/>
         <child link="rear_left_wheel"/>
-        <origin xyz="0.062 0.0725 0" rpy="-${pi/2} 0 0"/>
+        <origin xyz="${wheel_offset_rear} ${wheel_offset_side} 0" rpy="-${pi/2} 0 0"/>
         <axis xyz="0 0 1"/>
         <limit effort="${limit_effort}" velocity="${limit_velocity}"/>
@@ -110,5 +110,5 @@
         <parent link="base_link"/>
         <child link="rear_right_wheel"/>
-        <origin xyz="0.062 -0.0725 0" rpy="${pi/2} 0 0"/>
+        <origin xyz="${wheel_offset_rear} -${wheel_offset_side} 0" rpy="${pi/2} 0 0"/>
         <axis xyz="0 0 -1"/>
         <limit effort="${limit_effort}" velocity="${limit_velocity}"/>

Commit message: description/robot_core.xacro: Initial structure of bucket ladder
- Basic dimesions are correct, but the shapes are not, at least for the
  bucket ladder, and ideally, the ladder/lift is a frame and not solid.
- May replace later with at least two meshes for geometry

File: description/robot_core.xacro (robot description, xacro)
@@ -4,7 +4,14 @@
     <xacro:property name="limit_velocity" value="1" />
     <!-- Values in meters -->
+    <xacro:property name="buckets_length" value="0.254" /> <!-- depth -->
+    <xacro:property name="buckets_height" value="0.9144" />
+    <xacro:property name="buckets_width" value="0.1778" />
     <xacro:property name="chassis_length" value="0.8128" />
     <xacro:property name="chassis_height" value="0.0889" />
     <xacro:property name="chassis_width" value="0.3556" />
+    <xacro:property name="ladder_length" value="0.0508" /> <!-- depth -->
+    <xacro:property name="ladder_height" value="0.7874" />
+    <xacro:property name="ladder_width" value="${chassis_width}" />
+    <xacro:property name="ladder_offset" value="${-chassis_length/2 - buckets_length/2 - 0.0127}" />
     <xacro:property name="wheel_length" value="0.1016" />
     <xacro:property name="wheel_radius" value="0.1524" />
@@ -130,3 +137,53 @@
         </xacro:inertial_cylinder>
     </link>
+    <!-- Bucket Ladder Lift -->
+    <joint name="bucket_ladder_lift_joint" type="prismatic">
+        <parent link="base_link"/>
+        <child link="lift"/>
+        <limit lower="0"  upper="2"  velocity="0.1"  effort="${limit_effort}"  />
+        <axis xyz="0 0 1"/>
+        <origin xyz="${ladder_offset} 0 0" rpy="0 0 0"/>
+    </joint>
+    <link name="lift">
+        <collision>
+            <origin xyz="0 0 ${ladder_height/2}" rpy="0 0 0"/>
+            <geometry>
+                <box size="${ladder_length} ${ladder_width} ${ladder_height}"/>
+            </geometry>
+        </collision>
+        <visual>
+            <origin xyz="0 0 ${ladder_height/2}" rpy="0 0 0"/>
+            <geometry>
+                <box size="${ladder_length} ${ladder_width} ${ladder_height}"/>
+            </geometry>
+            <material name="green"/>
+        </visual>
+        <xacro:inertial_box mass="0.5" x="${ladder_length}" y="${ladder_width}" z="${ladder_height}">
+            <origin xyz="0 0 ${ladder_height/2}" rpy="0 0 0"/>
+        </xacro:inertial_box>
+    </link>
+    <!-- Bucket Ladder Buckets -->
+    <joint name="bucket_ladder_buckets_joint" type="continuous">
+        <parent link="lift"/>
+        <child link="buckets"/>
+        <axis xyz="0 0 1"/>
+    </joint>
+    <link name="buckets">
+        <collision>
+            <origin xyz="0 0 ${ladder_height/2}" rpy="0 0 0"/>
+            <geometry>
+                <box size="${buckets_length} ${buckets_width} ${buckets_height}"/>
+            </geometry>
+        </collision>
+        <visual>
+            <origin xyz="0 0 ${ladder_height/2}" rpy="0 0 0"/>
+            <geometry>
+                <box size="${buckets_length} ${buckets_width} ${buckets_height}"/>
+            </geometry>
+            <material name="red"/>
+        </visual>
+        <xacro:inertial_box mass="0.5" x="${buckets_length}" y="${buckets_width}" z="${buckets_height}">
+            <origin xyz="0 0 ${ladder_height/2}" rpy="0 0 0"/>
+        </xacro:inertial_box>
+    </link>
 </robot>

Commit message: description/robot_core.xacro: Switch to CAD wheel mesh from drawn

File: description/robot_core.xacro (robot description, xacro)
@@ -16,4 +16,6 @@
     <xacro:property name="wheel_length" value="0.1016" />
     <xacro:property name="wheel_radius" value="0.1524" />
+    <xacro:property name="wheel_mesh_file" value="package://osprey_ros/meshes/wheel.dae" />
+    <xacro:property name="wheel_mesh_scale" value="0.001 0.001 0.001" />
     <xacro:property name="wheel_offset_front" value="${-chassis_length/2 + 0.1778}" />
     <xacro:property name="wheel_offset_rear" value="${chassis_length/2 - 0.2286}" />
@@ -45,5 +47,5 @@
         <parent link="base_link"/>
         <child link="front_left_wheel"/>
-        <origin xyz="${wheel_offset_front} ${wheel_offset_side} 0" rpy="-${pi/2} 0 0"/>
+        <origin xyz="${wheel_offset_front} -${wheel_offset_side} 0" rpy="-${pi/2} 0 0"/>
         <axis xyz="0 0 1"/>
         <limit effort="${limit_effort}" velocity="${limit_velocity}"/>
@@ -56,8 +58,8 @@
         </collision>
         <visual>
+            <origin xyz="-${wheel_radius} ${wheel_radius} -${wheel_length/2}" rpy="${pi/2} 0 0"/>
             <geometry>
-                <cylinder length="${wheel_length}" radius="${wheel_radius}" />
+                <mesh filename="${wheel_mesh_file}" scale="${wheel_mesh_scale}" />
             </geometry>
-            <material name="yellow"/>
         </visual>
         <xacro:inertial_cylinder mass="0.1" length="${wheel_length}" radius="${wheel_radius}">
@@ -69,5 +71,5 @@
         <parent link="base_link"/>
         <child link="front_right_wheel"/>
-        <origin xyz="${wheel_offset_front} -${wheel_offset_side} 0" rpy="${pi/2} 0 0"/>
+        <origin xyz="${wheel_offset_front} ${wheel_offset_side} 0" rpy="${pi/2} 0 0"/>
         <axis xyz="0 0 -1"/>
         <limit effort="${limit_effort}" velocity="${limit_velocity}"/>
@@ -80,8 +82,8 @@
         </collision>
         <visual>
+            <origin xyz="-${wheel_radius} -${wheel_radius} ${wheel_length/2}" rpy="-${pi/2} 0 0"/>
             <geometry>
-                <cylinder length="${wheel_length}" radius="${wheel_radius}" />
+                <mesh filename="${wheel_mesh_file}" scale="${wheel_mesh_scale}" />
             </geometry>
-            <material name="yellow"/>
         </visual>
         <xacro:inertial_cylinder mass="0.1" length="${wheel_length}" radius="${wheel_radius}">
@@ -93,5 +95,5 @@
         <parent link="base_link"/>
         <child link="rear_left_wheel"/>
-        <origin xyz="${wheel_offset_rear} ${wheel_offset_side} 0" rpy="-${pi/2} 0 0"/>
+        <origin xyz="${wheel_offset_rear} -${wheel_offset_side} 0" rpy="-${pi/2} 0 0"/>
         <axis xyz="0 0 1"/>
         <limit effort="${limit_effort}" velocity="${limit_velocity}"/>
@@ -104,8 +106,8 @@
         </collision>
         <visual>
+            <origin xyz="-${wheel_radius} ${wheel_radius} -${wheel_length/2}" rpy="${pi/2} 0 0"/>
             <geometry>
-                <cylinder length="${wheel_length}" radius="${wheel_radius}" />
+                <mesh filename="${wheel_mesh_file}" scale="${wheel_mesh_scale}" />
             </geometry>
-            <material name="yellow"/>
         </visual>
         <xacro:inertial_cylinder mass="0.1" length="${wheel_length}" radius="${wheel_radius}">
@@ -117,5 +119,5 @@
         <parent link="base_link"/>
         <child link="rear_right_wheel"/>
-        <origin xyz="${wheel_offset_rear} -${wheel_offset_side} 0" rpy="${pi/2} 0 0"/>
+        <origin xyz="${wheel_offset_rear} ${wheel_offset_side} 0" rpy="${pi/2} 0 0"/>
         <axis xyz="0 0 -1"/>
         <limit effort="${limit_effort}" velocity="${limit_velocity}"/>
@@ -128,8 +130,8 @@
         </collision>
         <visual>
+            <origin xyz="-${wheel_radius} -${wheel_radius} ${wheel_length/2}" rpy="-${pi/2} 0 0"/>
             <geometry>
-                <cylinder length="${wheel_length}" radius="${wheel_radius}" />
+                <mesh filename="${wheel_mesh_file}" scale="${wheel_mesh_scale}" />
             </geometry>
-            <material name="yellow"/>
         </visual>
         <xacro:inertial_cylinder mass="0.1" length="${wheel_length}" radius="${wheel_radius}">

Commit message: description/robot_core.xacro: Switch to CAD chassis mesh from drawn

File: description/robot_core.xacro (robot description, xacro)
@@ -14,4 +14,5 @@
     <xacro:property name="ladder_width" value="${chassis_width}" />
     <xacro:property name="ladder_offset" value="${-chassis_length/2 - buckets_length/2 - 0.0127}" />
+    <xacro:property name="wheel_gap" value="0.0127" />
     <xacro:property name="wheel_length" value="0.1016" />
     <xacro:property name="wheel_radius" value="0.1524" />
@@ -20,5 +21,5 @@
     <xacro:property name="wheel_offset_front" value="${-chassis_length/2 + 0.1778}" />
     <xacro:property name="wheel_offset_rear" value="${chassis_length/2 - 0.2286}" />
-    <xacro:property name="wheel_offset_side" value="${wheel_length/2 + chassis_width/2 + 0.0127}" />
+    <xacro:property name="wheel_offset_side" value="${wheel_length/2 + chassis_width/2 + wheel_gap}" />
     <link name="base_link"></link>
     <!-- Main Body/Chassis -->
@@ -34,8 +35,8 @@
         </collision>
         <visual>
+            <origin xyz="-${chassis_length/2} ${chassis_length/2 - chassis_height - wheel_gap/2} -${chassis_width/2}" rpy="${pi/2} 0 0"/>
             <geometry>
-                <box size="${chassis_length} ${chassis_width} ${chassis_height}"/>
+                <mesh filename="package://osprey_ros/meshes/chassis.dae" scale="0.8 0.8 0.8" />
             </geometry>
-            <material name="blue"/>
         </visual>
         <xacro:inertial_box mass="0.5" x="${chassis_length}" y="${chassis_width}" z="${chassis_height}">

Commit message: description/robot_core.xacro: Added initial dump bucket using visual mesh

File: description/robot_core.xacro (robot description, xacro)
@@ -4,4 +4,7 @@
     <xacro:property name="limit_velocity" value="1" />
     <!-- Values in meters -->
+    <xacro:property name="bucket_length" value="0.3556" /> <!-- depth -->
+    <xacro:property name="bucket_height" value="0.254" />
+    <xacro:property name="bucket_width" value="0.254" />
     <xacro:property name="buckets_length" value="0.254" /> <!-- depth -->
     <xacro:property name="buckets_height" value="0.9144" />
@@ -35,5 +38,5 @@
         </collision>
         <visual>
-            <origin xyz="-${chassis_length/2} ${chassis_length/2 - chassis_height - wheel_gap/2} -${chassis_width/2}" rpy="${pi/2} 0 0"/>
+            <origin xyz="-${chassis_length/2 + chassis_height/2} ${chassis_length/2 - chassis_height - wheel_gap/2} -${chassis_width/2}" rpy="${pi/2} 0 0"/>
             <geometry>
                 <mesh filename="package://osprey_ros/meshes/chassis.dae" scale="0.8 0.8 0.8" />
@@ -190,3 +193,26 @@
         </xacro:inertial_box>
     </link>
+    <joint name="bucket_dump_joint" type="prismatic">
+        <parent link="base_link"/>
+        <child link="bucket"/>
+        <limit lower="0"  upper="2"  velocity="0.1"  effort="${limit_effort}"  />
+        <axis xyz="0 0 1"/>
+        <origin xyz="-${bucket_length/2} 0 ${bucket_height/2 + chassis_height}" rpy="0 0 0"/>
+    </joint>
+    <link name="bucket">
+        <collision>
+            <geometry>
+                <box size="${bucket_length} ${bucket_width} ${bucket_height}"/>
+            </geometry>
+        </collision>
+        <visual>
+            <origin xyz="-${bucket_length/2} ${bucket_length/2} -${chassis_height}" rpy="${pi/2} 0 0"/>
+            <geometry>
+                <mesh filename="package://osprey_ros/meshes/bucket_body.dae" scale="0.065 0.065 0.065" />
+            </geometry>
+        </visual>
+        <xacro:inertial_box mass="0.5" x="${bucket_length}" y="${bucket_width}" z="${bucket_height}">
+            <origin xyz="${chassis_length/2} 0 ${bucket_height/2}" rpy="0 0 0"/>
+        </xacro:inertial_box>
+    </link>
 </robot>

Commit message: description/robot_core.xacro: Switch to CAD buckets/gears mesh from drawn

File: description/robot_core.xacro (robot description, xacro)
@@ -183,7 +183,7 @@
         </collision>
         <visual>
-            <origin xyz="0 0 ${ladder_height/2}" rpy="0 0 0"/>
-            <geometry>
-                <box size="${buckets_length} ${buckets_width} ${buckets_height}"/>
+            <origin xyz="${buckets_length/1.25} ${ladder_width - wheel_gap*2.5} -${buckets_width/2}" rpy="${pi/2} -${pi/2} 0"/>
+            <geometry>
+                <mesh filename="package://osprey_ros/meshes/bucket_ladder_gears.dae" scale="0.9 0.9 0.9" />
             </geometry>
             <material name="red"/>

Commit message: description/robot_core.xacro: Switch to CAD lift frame mesh from drawn

File: description/robot_core.xacro (robot description, xacro)
@@ -159,7 +159,7 @@
         </collision>
         <visual>
-            <origin xyz="0 0 ${ladder_height/2}" rpy="0 0 0"/>
-            <geometry>
-                <box size="${ladder_length} ${ladder_width} ${ladder_height}"/>
+            <origin xyz="${buckets_length/1.25} ${ladder_width - wheel_gap*2.5} -${buckets_width/2}" rpy="${pi/2} -${pi/2} 0"/>
+            <geometry>
+                <mesh filename="package://osprey_ros/meshes/bucket_ladder_lift_frame.dae" scale="0.9 0.9 0.9" />
             </geometry>
             <material name="green"/>

Commit message: description/robot_core.xacro: Added bucket ladder guide frame joint w/ mesh

File: description/robot_core.xacro (robot description, xacro)
@@ -143,4 +143,30 @@
         </xacro:inertial_cylinder>
     </link>
+    <!-- Bucket Ladder Guide Frame -->
+    <joint name="bucket_ladder_frame_joint" type="prismatic">
+        <parent link="base_link"/>
+        <child link="guide_frame"/>
+        <limit lower="0"  upper="1"  velocity="0.1"  effort="${limit_effort}"  />
+        <axis xyz="0 0 1"/>
+        <origin xyz="${ladder_offset} 0 0" rpy="0 0 0"/>
+    </joint>
+    <link name="guide_frame">
+        <collision>
+            <origin xyz="0 0 ${ladder_height/2}" rpy="0 0 0"/>
+            <geometry>
+                <box size="${ladder_length} ${ladder_width} ${ladder_height}"/>
+            </geometry>
+        </collision>
+        <visual>
+            <origin xyz="${buckets_length/1.25} ${ladder_width - wheel_gap*2.5} -${buckets_width/2}" rpy="${pi/2} -${pi/2} 0"/>
+            <geometry>
+                <mesh filename="package://osprey_ros/meshes/bucket_ladder_guide_frame.dae" scale="0.9 0.9 0.9" />
+            </geometry>
+            <material name="green"/>
+        </visual>
+        <xacro:inertial_box mass="0.5" x="${ladder_length}" y="${ladder_width}" z="${ladder_height}">
+            <origin xyz="0 0 ${ladder_height/2}" rpy="0 0 0"/>
+        </xacro:inertial_box>
+    </link>
     <!-- Bucket Ladder Lift -->
     <joint name="bucket_ladder_lift_joint" type="prismatic">

Commit message: description/robot_core.xacro: Fix ladder orientation and alignment

File: description/robot_core.xacro (robot description, xacro)
@@ -7,4 +7,7 @@
     <xacro:property name="bucket_height" value="0.254" />
     <xacro:property name="bucket_width" value="0.254" />
+    <xacro:property name="bucket_ladder_scale" value="0.9 0.9 0.9" />
+    <xacro:property name="bucket_ladder_rpy" value="${pi/2} ${pi/2} 0" />
+    <xacro:property name="bucket_ladder_xyz" value="-${buckets_length/2 + ladder_length} ${ladder_width - wheel_gap*2.5} ${buckets_height - wheel_radius}" />
     <xacro:property name="buckets_length" value="0.254" /> <!-- depth -->
     <xacro:property name="buckets_height" value="0.9144" />
@@ -159,7 +162,7 @@
         </collision>
         <visual>
-            <origin xyz="${buckets_length/1.25} ${ladder_width - wheel_gap*2.5} -${buckets_width/2}" rpy="${pi/2} -${pi/2} 0"/>
-            <geometry>
-                <mesh filename="package://osprey_ros/meshes/bucket_ladder_guide_frame.dae" scale="0.9 0.9 0.9" />
+            <origin xyz="${bucket_ladder_xyz}" rpy="${bucket_ladder_rpy}"/>
+            <geometry>
+                <mesh filename="package://osprey_ros/meshes/bucket_ladder_guide_frame.dae" scale="${bucket_ladder_scale}" />
             </geometry>
             <material name="green"/>
@@ -185,7 +188,7 @@
         </collision>
         <visual>
-            <origin xyz="${buckets_length/1.25} ${ladder_width - wheel_gap*2.5} -${buckets_width/2}" rpy="${pi/2} -${pi/2} 0"/>
-            <geometry>
-                <mesh filename="package://osprey_ros/meshes/bucket_ladder_lift_frame.dae" scale="0.9 0.9 0.9" />
+            <origin xyz="${bucket_ladder_xyz}" rpy="${bucket_ladder_rpy}"/>
+            <geometry>
+                <mesh filename="package://osprey_ros/meshes/bucket_ladder_lift_frame.dae" scale="${bucket_ladder_scale}" />
             </geometry>
             <material name="green"/>
@@ -209,7 +212,7 @@
         </collision>
         <visual>
-            <origin xyz="${buckets_length/1.25} ${ladder_width - wheel_gap*2.5} -${buckets_width/2}" rpy="${pi/2} -${pi/2} 0"/>
-            <geometry>
-                <mesh filename="package://osprey_ros/meshes/bucket_ladder_gears.dae" scale="0.9 0.9 0.9" />
+            <origin xyz="${bucket_ladder_xyz}" rpy="${bucket_ladder_rpy}"/>
+            <geometry>
+                <mesh filename="package://osprey_ros/meshes/bucket_ladder_gears.dae" scale="${bucket_ladder_scale}" />
             </geometry>
             <material name="red"/>

Commit message: description/robot_core.xacro: Fixed dump bucket mesh filename change

File: description/robot_core.xacro (robot description, xacro)
@@ -238,5 +238,5 @@
             <origin xyz="-${bucket_length/2} ${bucket_length/2} -${chassis_height}" rpy="${pi/2} 0 0"/>
             <geometry>
-                <mesh filename="package://osprey_ros/meshes/bucket_body.dae" scale="0.065 0.065 0.065" />
+                <mesh filename="package://osprey_ros/meshes/dump_bucket_body.dae" scale="0.065 0.065 0.065" />
             </geometry>
         </visual>
