Commit message: description/robot_core.xacro: Fix Gazebo loading issue with mesh file paths
- Gazebo does not work with package:// file paths, only file://
  bad   package://osprey_ros
  good  file://$(find osprey_ros)

https://answers.ros.org/question/404423/whats-the-correct-way-to-load-mesh-files-in-gazebo-and-rviz/

File: description/robot_core.xacro (robot description, xacro)
@@ -23,5 +23,5 @@
     <xacro:property name="wheel_length" value="0.1016" />
     <xacro:property name="wheel_radius" value="0.1524" />
-    <xacro:property name="wheel_mesh_file" value="package://osprey_ros/meshes/wheel.dae" />
+    <xacro:property name="wheel_mesh_file" value="file://$(find osprey_ros)/meshes/wheel.dae" />
     <xacro:property name="wheel_mesh_scale" value="0.001 0.001 0.001" />
     <xacro:property name="wheel_offset_front" value="${-chassis_length/2 + 0.1778}" />
@@ -43,5 +43,5 @@
             <origin xyz="-${chassis_length/2 + chassis_height/2} ${chassis_length/2 - chassis_height - wheel_gap/2} -${chassis_width/2}" rpy="${pi/2} 0 0"/>
             <geometry>
-                <mesh filename="package://osprey_ros/meshes/chassis.dae" scale="0.8 0.8 0.8" />
+                <mesh filename="file://$(find osprey_ros)/meshes/chassis.dae" scale="0.8 0.8 0.8" />
             </geometry>
         </visual>
@@ -164,5 +164,5 @@
             <origin xyz="${bucket_ladder_xyz}" rpy="${bucket_ladder_rpy}"/>
             <geometry>
-                <mesh filename="package://osprey_ros/meshes/bucket_ladder_guide_frame.dae" scale="${bucket_ladder_scale}" />
+                <mesh filename="file://$(find osprey_ros)/meshes/bucket_ladder_guide_frame.dae" scale="${bucket_ladder_scale}" />
             </geometry>
             <material name="green"/>
@@ -190,5 +190,5 @@
             <origin xyz="${bucket_ladder_xyz}" rpy="${bucket_ladder_rpy}"/>
             <geometry>
-                <mesh filename="package://osprey_ros/meshes/bucket_ladder_lift_frame.dae" scale="${bucket_ladder_scale}" />
+                <mesh filename="file://$(find osprey_ros)/meshes/bucket_ladder_lift_frame.dae" scale="${bucket_ladder_scale}" />
             </geometry>
             <material name="green"/>
@@ -214,5 +214,5 @@
             <origin xyz="${bucket_ladder_xyz}" rpy="${bucket_ladder_rpy}"/>
             <geometry>
-                <mesh filename="package://osprey_ros/meshes/bucket_ladder_gears.dae" scale="${bucket_ladder_scale}" />
+                <mesh filename="file://$(find osprey_ros)/meshes/bucket_ladder_gears.dae" scale="${bucket_ladder_scale}" />
             </geometry>
             <material name="red"/>
@@ -238,5 +238,5 @@
             <origin xyz="-${bucket_length/2} ${bucket_length/2} -${chassis_height}" rpy="${pi/2} 0 0"/>
             <geometry>
-                <mesh filename="package://osprey_ros/meshes/dump_bucket_body.dae" scale="0.065 0.065 0.065" />
+                <mesh filename="file://$(find osprey_ros)/meshes/dump_bucket_body.dae" scale="0.065 0.065 0.065" />
             </geometry>
         </visual>

Commit message: description/robot_core.xacro: Lift up robot and change parents, fixes #2
- Lift up robot chassis by wheel radius
- Change parent of all elements except the chassis from base_link to chassis
  for all items that had base_link as the parent

File: description/robot_core.xacro (robot description, xacro)
@@ -32,4 +32,5 @@
     <joint name="chassis_joint" type="fixed">
         <parent link="base_link"/>
+        <origin xyz="0 0 ${wheel_radius}" rpy="0 0 0"/>
         <child link="chassis"/>
     </joint>
@@ -52,5 +53,5 @@
     <!-- Front Left Wheel -->
     <joint name="front_left_wheel_joint" type="continuous">
-        <parent link="base_link"/>
+        <parent link="chassis"/>
         <child link="front_left_wheel"/>
         <origin xyz="${wheel_offset_front} -${wheel_offset_side} 0" rpy="-${pi/2} 0 0"/>
@@ -76,5 +77,5 @@
     <!-- Front Right Wheel -->
     <joint name="front_right_wheel_joint" type="continuous">
-        <parent link="base_link"/>
+        <parent link="chassis"/>
         <child link="front_right_wheel"/>
         <origin xyz="${wheel_offset_front} ${wheel_offset_side} 0" rpy="${pi/2} 0 0"/>
@@ -100,5 +101,5 @@
     <!-- Rear Left Wheel -->
     <joint name="rear_left_wheel_joint" type="continuous">
-        <parent link="base_link"/>
+        <parent link="chassis"/>
         <child link="rear_left_wheel"/>
         <origin xyz="${wheel_offset_rear} -${wheel_offset_side} 0" rpy="-${pi/2} 0 0"/>
@@ -124,5 +125,5 @@
     <!-- Rear Right Wheel -->
     <joint name="rear_right_wheel_joint" type="continuous">
-        <parent link="base_link"/>
+        <parent link="chassis"/>
         <child link="rear_right_wheel"/>
         <origin xyz="${wheel_offset_rear} ${wheel_offset_side} 0" rpy="${pi/2} 0 0"/>
@@ -148,5 +149,5 @@
     <!-- Bucket Ladder Guide Frame -->
     <joint name="bucket_ladder_frame_joint" type="prismatic">
-        <parent link="base_link"/>
+        <parent link="chassis"/>
         <child link="guide_frame"/>
         <limit lower="0"  upper="1"  velocity="0.1"  effort="${limit_effort}"  />
@@ -174,5 +175,5 @@
     <!-- Bucket Ladder Lift -->
     <joint name="bucket_ladder_lift_joint" type="prismatic">
-        <parent link="base_link"/>
+        <parent link="chassis"/>
         <child link="lift"/>
         <limit lower="0"  upper="2"  velocity="0.1"  effort="${limit_effort}"  />
@@ -223,5 +224,5 @@
     </link>
     <joint name="bucket_dump_joint" type="prismatic">
-        <parent link="base_link"/>
+        <parent link="chassis"/>
         <child link="bucket"/>
         <limit lower="0"  upper="2"  velocity="0.1"  effort="${limit_effort}"  />

Commit message: description/robot_core.xacro: Gray material color for all mesh for gazebo
- Newer gazebo seems to require a material color otherwise it defaults to
  white, this is not an issue in gazebo classic or rviz2

File: description/robot_core.xacro (robot description, xacro)
@@ -46,4 +46,5 @@
                 <mesh filename="file://$(find osprey_ros)/meshes/chassis.dae" scale="0.8 0.8 0.8" />
             </geometry>
+            <material name="gray"/>
         </visual>
         <xacro:inertial_box mass="0.5" x="${chassis_length}" y="${chassis_width}" z="${chassis_height}">
@@ -70,4 +71,5 @@
                 <mesh filename="${wheel_mesh_file}" scale="${wheel_mesh_scale}" />
             </geometry>
+            <material name="gray"/>
         </visual>
         <xacro:inertial_cylinder mass="0.1" length="${wheel_length}" radius="${wheel_radius}">
@@ -94,4 +96,5 @@
                 <mesh filename="${wheel_mesh_file}" scale="${wheel_mesh_scale}" />
             </geometry>
+            <material name="gray"/>
         </visual>
         <xacro:inertial_cylinder mass="0.1" length="${wheel_length}" radius="${wheel_radius}">
@@ -118,4 +121,5 @@
                 <mesh filename="${wheel_mesh_file}" scale="${wheel_mesh_scale}" />
             </geometry>
+            <material name="gray"/>
         </visual>
         <xacro:inertial_cylinder mass="0.1" length="${wheel_length}" radius="${wheel_radius}">
@@ -142,4 +146,5 @@
                 <mesh filename="${wheel_mesh_file}" scale="${wheel_mesh_scale}" />
             </geometry>
+            <material name="gray"/>
         </visual>
         <xacro:inertial_cylinder mass="0.1" length="${wheel_length}" radius="${wheel_radius}">
@@ -161,4 +166,5 @@
                 <box size="${ladder_length} ${ladder_width} ${ladder_height}"/>
             </geometry>
+            <material name="gray"/>
         </collision>
         <visual>
@@ -167,5 +173,5 @@
                 <mesh filename="file://$(find osprey_ros)/meshes/bucket_ladder_guide_frame.dae" scale="${bucket_ladder_scale}" />
             </geometry>
-            <material name="green"/>
+            <material name="gray"/>
         </visual>
         <xacro:inertial_box mass="0.5" x="${ladder_length}" y="${ladder_width}" z="${ladder_height}">
@@ -193,5 +199,5 @@
                 <mesh filename="file://$(find osprey_ros)/meshes/bucket_ladder_lift_frame.dae" scale="${bucket_ladder_scale}" />
             </geometry>
-            <material name="green"/>
+            <material name="gray"/>
         </visual>
         <xacro:inertial_box mass="0.5" x="${ladder_length}" y="${ladder_width}" z="${ladder_height}">
@@ -217,5 +223,5 @@
                 <mesh filename="file://$(find osprey_ros)/meshes/bucket_ladder_gears.dae" scale="${bucket_ladder_scale}" />
             </geometry>
-            <material name="red"/>
+            <material name="gray"/>
         </visual>
         <xacro:inertial_box mass="0.5" x="${buckets_length}" y="${buckets_width}" z="${buckets_height}">
@@ -241,4 +247,5 @@
                 <mesh filename="file://$(find osprey_ros)/meshes/dump_bucket_body.dae" scale="0.065 0.065 0.065" />
             </geometry>
+            <material name="gray"/>
         </visual>
         <xacro:inertial_box mass="0.5" x="${bucket_length}" y="${bucket_width}" z="${bucket_height}">

Commit message: description/robot_core.xacro: Correct bucket lift parent remove origin
- Corrected the bucket lift parent to guide_frame, the frame that houses
  the entire bucket ladder system, lift and buckets
- Removed origin from bucket ladder lift joint

File: description/robot_core.xacro (robot description, xacro)
@@ -181,9 +181,8 @@
     <!-- Bucket Ladder Lift -->
     <joint name="bucket_ladder_lift_joint" type="prismatic">
-        <parent link="chassis"/>
+        <parent link="guide_frame"/>
         <child link="lift"/>
         <limit lower="0"  upper="2"  velocity="0.1"  effort="${limit_effort}"  />
         <axis xyz="0 0 1"/>
-        <origin xyz="${ladder_offset} 0 0" rpy="0 0 0"/>
     </joint>
     <link name="lift">

Commit message: description/robot_core.xacro: Change ladder frame joint type and some limts
- Changed the ladder frame joint type from prismatic to revolute, so it
  moves on a hinged axis, the Y axis.
- Updated the ladder frame joint limits to move within a range of 90° to 60°
  extended to retracted
- Updated the ladder lift joint limits to move within a range of -0.5 to 0
  down to up

File: description/robot_core.xacro (robot description, xacro)
@@ -153,9 +153,9 @@
     </link>
     <!-- Bucket Ladder Guide Frame -->
-    <joint name="bucket_ladder_frame_joint" type="prismatic">
+    <joint name="bucket_ladder_frame_joint" type="revolute">
         <parent link="chassis"/>
         <child link="guide_frame"/>
-        <limit lower="0"  upper="1"  velocity="0.1"  effort="${limit_effort}"  />
-        <axis xyz="0 0 1"/>
+        <limit lower="0"  upper="0.523598775598"  velocity="0.1"  effort="${limit_effort}"  />
+        <axis xyz="0 1 0"/>
         <origin xyz="${ladder_offset} 0 0" rpy="0 0 0"/>
     </joint>
@@ -183,5 +183,5 @@
         <parent link="guide_frame"/>
         <child link="lift"/>
-        <limit lower="0"  upper="2"  velocity="0.1"  effort="${limit_effort}"  />
+        <limit lower="-0.5"  upper="0"  velocity="0.1"  effort="${limit_effort}"  />
         <axis xyz="0 0 1"/>
     </joint>

Commit message: description/robot_core.xacro: Tweak mass & limits for ladder frame & lift

File: description/robot_core.xacro (robot description, xacro)
@@ -175,5 +175,5 @@
             <material name="gray"/>
         </visual>
-        <xacro:inertial_box mass="0.25" x="${ladder_length}" y="${ladder_width}" z="${ladder_height}">
+        <xacro:inertial_box mass="0.75" x="${ladder_length}" y="${ladder_width}" z="${ladder_height}">
             <origin xyz="0 0 ${ladder_height/2}" rpy="0 0 0"/>
         </xacro:inertial_box>
@@ -183,5 +183,5 @@
         <parent link="guide_frame"/>
         <child link="lift"/>
-        <limit lower="-0.5"  upper="0"  velocity="0.1"  effort="${limit_effort}"  />
+        <limit lower="-0.35"  upper="0"  velocity="0.1"  effort="${limit_effort}"  />
         <axis xyz="0 0 1"/>
     </joint>
@@ -200,5 +200,5 @@
             <material name="gray"/>
         </visual>
-        <xacro:inertial_box mass="0.1" x="${ladder_length}" y="${ladder_width}" z="${ladder_height}">
+        <xacro:inertial_box mass="0.01" x="${ladder_length}" y="${ladder_width}" z="${ladder_height}">
             <origin xyz="0 0 ${ladder_height/2}" rpy="0 0 0"/>
         </xacro:inertial_box>

Commit message: description/robot_core.xacro: Flip backward robot model correct direction
- The robot model was backwards, and when moving foward was going -X vs +X,
  heading towards quandrants II and III instead of I and IV.
- Modified some origins and other values to correct physics, which needs
  work the masses and inertia values are likely not accurate

File: description/robot_core.xacro (robot description, xacro)
@@ -7,7 +7,7 @@
     <xacro:property name="bucket_height" value="0.254" />
     <xacro:property name="bucket_width" value="0.254" />
-    <xacro:property name="bucket_ladder_scale" value="0.9 0.9 0.9" />
-    <xacro:property name="bucket_ladder_rpy" value="${pi/2} ${pi/2} 0" />
-    <xacro:property name="bucket_ladder_xyz" value="-${buckets_length/2 + ladder_length} ${ladder_width - wheel_gap*2.5} ${buckets_height - wheel_radius}" />
+    <xacro:property name="bucket_ladder_scale" value="1 1 1" />
+    <xacro:property name="bucket_ladder_rpy" value="-${pi/2} ${pi/2} 0" />
+    <xacro:property name="bucket_ladder_xyz" value="${buckets_length} -${ladder_width + wheel_gap/4} ${buckets_height - chassis_height/1.25}" />
     <xacro:property name="buckets_length" value="0.254" /> <!-- depth -->
     <xacro:property name="buckets_height" value="0.9144" />
@@ -19,5 +19,6 @@
     <xacro:property name="ladder_height" value="0.7874" />
     <xacro:property name="ladder_width" value="${chassis_width}" />
-    <xacro:property name="ladder_offset" value="${-chassis_length/2 - buckets_length/2 - 0.0127}" />
+    <xacro:property name="ladder_offset" value="${chassis_length/2 + buckets_width/10}" />
+    <xacro:property name="ladder_xyz" value="${buckets_length} -${ladder_width + wheel_gap/4} ${buckets_height - chassis_height/2}" />
     <xacro:property name="wheel_gap" value="0.0127" />
     <xacro:property name="wheel_length" value="0.1016" />
@@ -42,5 +43,5 @@
         </collision>
         <visual>
-            <origin xyz="-${chassis_length/2 + chassis_height/2} ${chassis_length/2 - chassis_height - wheel_gap/2} -${chassis_width/2}" rpy="${pi/2} 0 0"/>
+            <origin xyz="-${chassis_length/2} ${chassis_length/2 - chassis_height - wheel_gap/2} -${chassis_width/2}" rpy="${pi/2} 0 0"/>
             <geometry>
                 <mesh filename="file://$(find osprey_ros)/meshes/chassis.dae" scale="0.8 0.8 0.8" />
@@ -49,5 +50,5 @@
         </visual>
         <xacro:inertial_box mass="2" x="${chassis_length}" y="${chassis_width}" z="${chassis_height}">
-            <origin xyz="${chassis_length/2} 0 0" rpy="0 0 0"/>
+            <origin xyz="0 0 0" rpy="0 0 0"/>
         </xacro:inertial_box>
     </link>
@@ -56,5 +57,5 @@
         <parent link="chassis"/>
         <child link="front_left_wheel"/>
-        <origin xyz="${wheel_offset_front} -${wheel_offset_side} 0" rpy="-${pi/2} 0 0"/>
+        <origin xyz="${wheel_offset_front} ${wheel_offset_side} 0" rpy="-${pi/2} 0 0"/>
         <axis xyz="0 0 1"/>
         <limit effort="${limit_effort}" velocity="${limit_velocity}"/>
@@ -67,5 +68,5 @@
         </collision>
         <visual>
-            <origin xyz="-${wheel_radius} ${wheel_radius} -${wheel_length/2}" rpy="${pi/2} 0 0"/>
+            <origin xyz="-${wheel_radius} -${wheel_radius} ${wheel_length/2}" rpy="-${pi/2} 0 0"/>
             <geometry>
                 <mesh filename="${wheel_mesh_file}" scale="${wheel_mesh_scale}" />
@@ -81,5 +82,5 @@
         <parent link="chassis"/>
         <child link="front_right_wheel"/>
-        <origin xyz="${wheel_offset_front} ${wheel_offset_side} 0" rpy="${pi/2} 0 0"/>
+        <origin xyz="${wheel_offset_front} -${wheel_offset_side} 0" rpy="${pi/2} 0 0"/>
         <axis xyz="0 0 -1"/>
         <limit effort="${limit_effort}" velocity="${limit_velocity}"/>
@@ -92,5 +93,5 @@
         </collision>
         <visual>
-            <origin xyz="-${wheel_radius} -${wheel_radius} ${wheel_length/2}" rpy="-${pi/2} 0 0"/>
+            <origin xyz="-${wheel_radius} ${wheel_radius} -${wheel_length/2}" rpy="${pi/2} 0 0"/>
             <geometry>
                 <mesh filename="${wheel_mesh_file}" scale="${wheel_mesh_scale}" />
@@ -106,5 +107,5 @@
         <parent link="chassis"/>
         <child link="rear_left_wheel"/>
-        <origin xyz="${wheel_offset_rear} -${wheel_offset_side} 0" rpy="-${pi/2} 0 0"/>
+        <origin xyz="${wheel_offset_rear} ${wheel_offset_side} 0" rpy="-${pi/2} 0 0"/>
         <axis xyz="0 0 1"/>
         <limit effort="${limit_effort}" velocity="${limit_velocity}"/>
@@ -117,5 +118,5 @@
         </collision>
         <visual>
-            <origin xyz="-${wheel_radius} ${wheel_radius} -${wheel_length/2}" rpy="${pi/2} 0 0"/>
+            <origin xyz="-${wheel_radius} -${wheel_radius} ${wheel_length/2}" rpy="-${pi/2} 0 0"/>
             <geometry>
                 <mesh filename="${wheel_mesh_file}" scale="${wheel_mesh_scale}" />
@@ -131,5 +132,5 @@
         <parent link="chassis"/>
         <child link="rear_right_wheel"/>
-        <origin xyz="${wheel_offset_rear} ${wheel_offset_side} 0" rpy="${pi/2} 0 0"/>
+        <origin xyz="${wheel_offset_rear} -${wheel_offset_side} 0" rpy="${pi/2} 0 0"/>
         <axis xyz="0 0 -1"/>
         <limit effort="${limit_effort}" velocity="${limit_velocity}"/>
@@ -142,5 +143,5 @@
         </collision>
         <visual>
-            <origin xyz="-${wheel_radius} -${wheel_radius} ${wheel_length/2}" rpy="-${pi/2} 0 0"/>
+            <origin xyz="-${wheel_radius} ${wheel_radius} -${wheel_length/2}" rpy="${pi/2} 0 0"/>
             <geometry>
                 <mesh filename="${wheel_mesh_file}" scale="${wheel_mesh_scale}" />
@@ -156,5 +157,5 @@
         <parent link="chassis"/>
         <child link="guide_frame"/>
-        <limit lower="0"  upper="0.523598775598"  velocity="0.1"  effort="${limit_effort}"  />
+        <limit lower="0"  upper="-0.523598775598"  velocity="0.1"  effort="${limit_effort}"  />
         <axis xyz="0 1 0"/>
         <origin xyz="${ladder_offset} 0 0" rpy="0 0 0"/>
@@ -194,5 +195,5 @@
         </collision>
         <visual>
-            <origin xyz="${bucket_ladder_xyz}" rpy="${bucket_ladder_rpy}"/>
+            <origin xyz="${ladder_xyz}" rpy="${bucket_ladder_rpy}"/>
             <geometry>
                 <mesh filename="file://$(find osprey_ros)/meshes/bucket_ladder_lift_frame.dae" scale="${bucket_ladder_scale}" />
@@ -218,5 +219,5 @@
         </collision>
         <visual>
-            <origin xyz="${bucket_ladder_xyz}" rpy="${bucket_ladder_rpy}"/>
+            <origin xyz="${ladder_xyz}" rpy="${bucket_ladder_rpy}"/>
             <geometry>
                 <mesh filename="file://$(find osprey_ros)/meshes/bucket_ladder_gears.dae" scale="${bucket_ladder_scale}" />
@@ -233,5 +234,5 @@
         <limit lower="0"  upper="2"  velocity="0.1"  effort="${limit_effort}"  />
         <axis xyz="0 0 1"/>
-        <origin xyz="-${bucket_length/2} 0 ${bucket_height/2 + chassis_height}" rpy="0 0 0"/>
+        <origin xyz="${bucket_length/2} 0 ${bucket_height/2 + chassis_height}" rpy="0 0 0"/>
     </joint>
     <link name="bucket">
@@ -242,5 +243,5 @@
         </collision>
         <visual>
-            <origin xyz="-${bucket_length/2} ${bucket_length/2} -${chassis_height}" rpy="${pi/2} 0 0"/>
+            <origin xyz="${bucket_length/2} -${bucket_width/1.6} -${chassis_height}" rpy="${pi/2} 0 ${pi}"/>
             <geometry>
                 <mesh filename="file://$(find osprey_ros)/meshes/dump_bucket_body.dae" scale="0.065 0.065 0.065" />
