Commit message: description/robot_core.xacro: Adjust mass values, add var for wheel mass

File: description/robot_core.xacro (robot description, xacro)
@@ -2,5 +2,5 @@
 <robot xmlns:xacro="http://www.ros.org/wiki/xacro">
     <xacro:property name="limit_effort" value="100" />
-    <xacro:property name="limit_velocity" value="1" />
+    <xacro:property name="limit_velocity" value="10" />
     <!-- Values in meters -->
     <xacro:property name="bucket_length" value="0.3556" /> <!-- depth -->
@@ -24,4 +24,5 @@
     <xacro:property name="wheel_length" value="0.1016" />
     <xacro:property name="wheel_radius" value="0.1524" />
+    <xacro:property name="wheel_mass" value="0.0624" />
     <xacro:property name="wheel_mesh_file" value="file://$(find osprey_ros)/meshes/wheel.dae" />
     <xacro:property name="wheel_mesh_scale" value="0.001 0.001 0.001" />
@@ -49,5 +50,5 @@
             <material name="gray"/>
         </visual>
-        <xacro:inertial_box mass="2" x="${chassis_length}" y="${chassis_width}" z="${chassis_height}">
+        <xacro:inertial_box mass="2.5" x="${chassis_length}" y="${chassis_width}" z="${chassis_height}">
             <origin xyz="0 0 0" rpy="0 0 0"/>
         </xacro:inertial_box>
@@ -74,5 +75,5 @@
             <material name="gray"/>
         </visual>
-        <xacro:inertial_cylinder mass="0.5" length="${wheel_length}" radius="${wheel_radius}">
+        <xacro:inertial_cylinder mass="${wheel_mass}" length="${wheel_length}" radius="${wheel_radius}">
             <origin xyz="0 0 0" rpy="0 0 0"/>
         </xacro:inertial_cylinder>
@@ -99,5 +100,5 @@
             <material name="gray"/>
         </visual>
-        <xacro:inertial_cylinder mass="0.5" length="${wheel_length}" radius="${wheel_radius}">
+        <xacro:inertial_cylinder mass="${wheel_mass}" length="${wheel_length}" radius="${wheel_radius}">
             <origin xyz="0 0 0" rpy="0 0 0"/>
         </xacro:inertial_cylinder>
@@ -124,5 +125,5 @@
             <material name="gray"/>
         </visual>
-        <xacro:inertial_cylinder mass="0.5" length="${wheel_length}" radius="${wheel_radius}">
+        <xacro:inertial_cylinder mass="${wheel_mass}" length="${wheel_length}" radius="${wheel_radius}">
             <origin xyz="0 0 0" rpy="0 0 0"/>
         </xacro:inertial_cylinder>
@@ -149,5 +150,5 @@
             <material name="gray"/>
         </visual>
-        <xacro:inertial_cylinder mass="0.5" length="${wheel_length}" radius="${wheel_radius}">
+        <xacro:inertial_cylinder mass="${wheel_mass}" length="${wheel_length}" radius="${wheel_radius}">
             <origin xyz="0 0 0" rpy="0 0 0"/>
         </xacro:inertial_cylinder>
@@ -176,5 +177,5 @@
             <material name="gray"/>
         </visual>
-        <xacro:inertial_box mass="0.75" x="${ladder_length}" y="${ladder_width}" z="${ladder_height}">
+        <xacro:inertial_box mass="0.05" x="${ladder_length}" y="${ladder_width}" z="${ladder_height}">
             <origin xyz="0 0 ${ladder_height/2}" rpy="0 0 0"/>
         </xacro:inertial_box>
@@ -249,5 +250,5 @@
             <material name="gray"/>
         </visual>
-        <xacro:inertial_box mass="0.5" x="${bucket_length}" y="${bucket_width}" z="${bucket_height}">
+        <xacro:inertial_box mass="0.1" x="${bucket_length}" y="${bucket_width}" z="${bucket_height}">
             <origin xyz="${chassis_length/2} 0 ${bucket_height/2}" rpy="0 0 0"/>
         </xacro:inertial_box>

Commit message: description/robot_core.xacro: Invert frame joint limits, correct order

File: description/robot_core.xacro (robot description, xacro)
@@ -158,5 +158,5 @@
         <parent link="chassis"/>
         <child link="guide_frame"/>
-        <limit lower="0"  upper="-0.523598775598"  velocity="0.1"  effort="${limit_effort}"  />
+        <limit lower="-0.523598775598"  upper="0"  velocity="0.1"  effort="${limit_effort}"  />
         <axis xyz="0 1 0"/>
         <origin xyz="${ladder_offset} 0 0" rpy="0 0 0"/>

Commit message: description/robot_core.xacro: Added rplidar to top of bucket ladder frame

File: description/robot_core.xacro (robot description, xacro)
@@ -21,4 +21,7 @@
     <xacro:property name="ladder_offset" value="${chassis_length/2 + buckets_width/10}" />
     <xacro:property name="ladder_xyz" value="${buckets_length} -${ladder_width + wheel_gap/4} ${buckets_height - chassis_height/2}" />
+    <xacro:property name="lidar_length" value="0.12954" />
+    <xacro:property name="lidar_height" value="0.07874" />
+    <xacro:property name="lidar_width" value="0.09906" />
     <xacro:property name="wheel_gap" value="0.0127" />
     <xacro:property name="wheel_length" value="0.1016" />
@@ -254,3 +257,26 @@
         </xacro:inertial_box>
     </link>
+    <joint name="lidar_joint" type="fixed">
+        <parent link="guide_frame"/>
+        <child link="lidar"/>
+        <axis xyz="0 0 0"/>
+        <origin xyz="${ladder_length/1.5} 0 ${ladder_height + lidar_height}" rpy="0 0 0"/>
+    </joint>
+    <link name="lidar">
+        <collision>
+            <geometry>
+                <box size="${lidar_length} ${lidar_width} ${lidar_height}"/>
+            </geometry>
+        </collision>
+        <visual>
+            <origin xyz="0 0 0" rpy="0 0 0"/>
+            <geometry>
+                <mesh filename="file://$(find osprey_ros)/meshes/rplidar.dae" scale="1 1 1" />
+            </geometry>
+            <material name="gray"/>
+        </visual>
+        <xacro:inertial_box mass="0.0001" x="${lidar_length}" y="${lidar_width}" z="${ladder_height}">
+            <origin xyz="${lidar_length/2} ${lidar_width/2} ${ladder_height/2}" rpy="0 0 0"/>
+        </xacro:inertial_box>
+    </link>
 </robot>

Commit message: description/robot_core.xacro: Add simulated lidar for gazebo

File: description/robot_core.xacro (robot description, xacro)
@@ -260,5 +260,5 @@
         <parent link="guide_frame"/>
         <child link="lidar"/>
-        <axis xyz="0 0 0"/>
+        <axis xyz="0 0 1"/>
         <origin xyz="${ladder_length/1.5} 0 ${ladder_height + lidar_height}" rpy="0 0 0"/>
     </joint>
@@ -280,3 +280,27 @@
         </xacro:inertial_box>
     </link>
+    <gazebo reference="lidar">
+        <sensor name="lidar_sensor" type="gpu_lidar">
+            <pose>0 0 0 0 0 0</pose>
+            <topic>lidar</topic>
+            <update_rate>10</update_rate>
+            <lidar>
+                <scan>
+                    <horizontal>
+                        <samples>360</samples>
+                        <min_angle>-3.14</min_angle>
+                        <max_angle>3.14</max_angle>
+                        <resolution>1</resolution>
+                    </horizontal>
+                </scan>
+                <range>
+                    <min>0.3</min>
+                    <max>12</max>
+                    <resolution>0.01</resolution>
+                </range>
+            </lidar>
+            <always_on>1</always_on>
+            <visualize>true</visualize>
+        </sensor>
+    </gazebo>
 </robot>

Commit message: description/robot_core.xacro: Added base_footprint{,_joint} link & joint
- Added base_footprint_joint joint with base_footprint link as a child for
  use with slam_toolbox

File: description/robot_core.xacro (robot description, xacro)
@@ -34,4 +34,11 @@
     <xacro:property name="wheel_offset_side" value="${wheel_length/2 + chassis_width/2 + wheel_gap}" />
     <link name="base_link"></link>
+    <joint name="base_footprint_joint" type="fixed">
+        <parent link="base_link"/>
+        <child link="base_footprint"/>
+    </joint>
+    <link name="base_footprint">
+        <parent link="base_link"/>
+    </link>
     <!-- Main Body/Chassis -->
     <joint name="chassis_joint" type="fixed">

Commit message: description/robot_core.xacro: Added collision multiplier enlarge buffer zone
- Added a collision multiplier value of 2 to increase lengths and widths
  to enlarge the buffer zone around the robot

File: description/robot_core.xacro (robot description, xacro)
@@ -1,4 +1,5 @@
 <?xml version="1.0"?>
 <robot xmlns:xacro="http://www.ros.org/wiki/xacro">
+    <xacro:property name="collision_multiplier" value="2" />
     <xacro:property name="limit_effort" value="100" />
     <xacro:property name="limit_velocity" value="10" />
@@ -50,5 +51,5 @@
         <collision>
             <geometry>
-                <box size="${chassis_length} ${chassis_width} ${chassis_height}"/>
+                <box size="${chassis_length * collision_multiplier} ${chassis_width * collision_multiplier} ${chassis_height}"/>
             </geometry>
         </collision>
@@ -75,5 +76,5 @@
         <collision>
             <geometry>
-                <cylinder length="${wheel_length}" radius="${wheel_radius}" />
+                <cylinder length="${wheel_length * collision_multiplier}" radius="${wheel_radius}" />
             </geometry>
         </collision>
@@ -100,5 +101,5 @@
         <collision>
             <geometry>
-                <cylinder length="${wheel_length}" radius="${wheel_radius}" />
+                <cylinder length="${wheel_length * collision_multiplier}" radius="${wheel_radius}" />
             </geometry>
         </collision>
@@ -125,5 +126,5 @@
         <collision>
             <geometry>
-                <cylinder length="${wheel_length}" radius="${wheel_radius}" />
+                <cylinder length="${wheel_length * collision_multiplier}" radius="${wheel_radius}" />
             </geometry>
         </collision>
@@ -150,5 +151,5 @@
         <collision>
             <geometry>
-                <cylinder length="${wheel_length}" radius="${wheel_radius}" />
+                <cylinder length="${wheel_length * collision_multiplier}" radius="${wheel_radius}" />
             </geometry>
         </collision>
@@ -176,5 +177,5 @@
             <origin xyz="0 0 ${ladder_height/2}" rpy="0 0 0"/>
             <geometry>
-                <box size="${ladder_length} ${ladder_width} ${ladder_height}"/>
+                <box size="${ladder_length * collision_multiplier} ${ladder_width * collision_multiplier} ${ladder_height}"/>
             </geometry>
             <material name="gray"/>
@@ -226,5 +227,5 @@
             <origin xyz="0 0 ${ladder_height/2}" rpy="0 0 0"/>
             <geometry>
-                <box size="${buckets_length} ${buckets_width} ${buckets_height}"/>
+                <box size="${buckets_length * collision_multiplier} ${buckets_width * collision_multiplier} ${buckets_height}"/>
             </geometry>
         </collision>

Commit message: description/robot_core.xacro: Reduce collision zone multiplier

File: description/robot_core.xacro (robot description, xacro)
@@ -1,5 +1,5 @@
 <?xml version="1.0"?>
 <robot xmlns:xacro="http://www.ros.org/wiki/xacro">
-    <xacro:property name="collision_multiplier" value="2" />
+    <xacro:property name="collision_multiplier" value="1.5" />
     <xacro:property name="limit_effort" value="100" />
     <xacro:property name="limit_velocity" value="10" />

Commit message: description/robot_core.xacro: Added joint and link for 3d camera

File: description/robot_core.xacro (robot description, xacro)
@@ -290,3 +290,23 @@
         </xacro:inertial_box>
     </link>
+    <!-- 3D Camera -->
+    <joint name="depth_camera_joint" type="fixed">
+        <parent link="chassis"/>
+        <child link="depth_camera"/>
+        <origin xyz="${buckets_length/2 + chassis_length/2} 0 0" rpy="0 0 0"/>
+    </joint>
+    <link name="depth_camera">
+        <visual>
+            <geometry>
+                <box size="0.010 0.03 0.03"/>
+            </geometry>
+            <material name="black"/>
+        </visual>
+        <visual>
+            <origin xyz="0 0 0"/>
+            <geometry>
+                <cylinder radius="0.002" length="0.1"/>
+            </geometry>
+        </visual>
+    </link>
 </robot>

Commit message: description/robot_core.xacro: Change lidar color to black from gray

File: description/robot_core.xacro (robot description, xacro)
@@ -284,5 +284,5 @@
                 <mesh filename="file://$(find osprey_ros)/meshes/rplidar.dae" scale="1 1 1" />
             </geometry>
-            <material name="gray"/>
+            <material name="black"/>
         </visual>
         <xacro:inertial_box mass="0.0001" x="${lidar_length}" y="${lidar_width}" z="${ladder_height}">
