Commit message: description/robot24_ros2_control.xacro: Added bucket_joint position joint

File: description/robot24_ros2_control.xacro (robot description, xacro)
@@ -57,4 +57,13 @@
             </state_interface>
         </joint>
+        <joint name="bucket_joint">
+            <command_interface name="position">
+                <param name="min">-1</param>
+                <param name="max">1</param>
+            </command_interface>
+            <state_interface name="position">
+                <param name="initial_value">0</param>
+            </state_interface>
+        </joint>
     </ros2_control>
   </xacro:macro>
