Commit message: description/robot24_core.xacro: Corrected & aligned chassis & wheels sizes
- Modified visual orgins of meshes, now that they are properly centered it
  simplifies usage and less translations
- Corrected wheel offsets to match with chassis holes
- Made mesh scale of chassis and wheels the same

File: description/robot24_core.xacro (robot description, xacro)
@@ -7,12 +7,12 @@
     <xacro:property name="chassis_height" value="0.0889" />
     <xacro:property name="chassis_width" value="0.3556" />
+    <xacro:property name="mesh_scale" value="0.001 0.001 0.001" />
     <xacro:property name="wheel_gap" value="0.0127" />
     <xacro:property name="wheel_length" value="0.1016" />
-    <xacro:property name="wheel_radius" value="0.1524" />
+    <xacro:property name="wheel_radius" value="0.1397" />
     <xacro:property name="wheel_mass" value="0.0624" />
     <xacro:property name="wheel_mesh_file" value="file://$(find osprey_ros)/meshes/robot24/wheel.dae" />
-    <xacro:property name="wheel_mesh_scale" value="0.001 0.001 0.001" />
-    <xacro:property name="wheel_offset_front" value="${-chassis_length/2 + 0.1778}" />
-    <xacro:property name="wheel_offset_rear" value="${chassis_length/2 - 0.2286}" />
+    <xacro:property name="wheel_offset_front" value="${chassis_length/2 - 0.1024}" />
+    <xacro:property name="wheel_offset_rear" value="${-chassis_length/2 + 0.1024}" />
     <xacro:property name="wheel_offset_side" value="${wheel_length/2 + chassis_width/2 + wheel_gap}" />
     <link name="base_link"></link>
@@ -37,7 +37,6 @@
         </collision>
         <visual>
-            <origin xyz="-${chassis_length/2} ${chassis_length/2 - chassis_height - wheel_gap/2} -${chassis_width/2}" rpy="${pi/2} 0 0"/>
             <geometry>
-                <mesh filename="file://$(find osprey_ros)/meshes/robot24/chassis.dae" scale="0.8 0.8 0.8" />
+                <mesh filename="file://$(find osprey_ros)/meshes/robot24/chassis.dae" scale="${mesh_scale}" />
             </geometry>
             <material name="gray"/>
@@ -62,7 +61,7 @@
         </collision>
         <visual>
-            <origin xyz="-${wheel_radius} -${wheel_radius} ${wheel_length/2}" rpy="-${pi/2} 0 0"/>
+            <origin xyz="0 0 ${wheel_length/2}" rpy="-${pi/2} 0 0"/>
             <geometry>
-                <mesh filename="${wheel_mesh_file}" scale="${wheel_mesh_scale}" />
+                <mesh filename="${wheel_mesh_file}" scale="${mesh_scale}" />
             </geometry>
             <material name="gray"/>
@@ -87,7 +86,7 @@
         </collision>
         <visual>
-            <origin xyz="-${wheel_radius} ${wheel_radius} -${wheel_length/2}" rpy="${pi/2} 0 0"/>
+            <origin xyz="0 0 ${wheel_length/2}" rpy="-${pi/2} 0 0"/>
             <geometry>
-                <mesh filename="${wheel_mesh_file}" scale="${wheel_mesh_scale}" />
+                <mesh filename="${wheel_mesh_file}" scale="${mesh_scale}" />
             </geometry>
             <material name="gray"/>
@@ -112,7 +111,7 @@
         </collision>
         <visual>
-            <origin xyz="-${wheel_radius} -${wheel_radius} ${wheel_length/2}" rpy="-${pi/2} 0 0"/>
+            <origin xyz="0 0 ${wheel_length/2}" rpy="-${pi/2} 0 0"/>
             <geometry>
-                <mesh filename="${wheel_mesh_file}" scale="${wheel_mesh_scale}" />
+                <mesh filename="${wheel_mesh_file}" scale="${mesh_scale}" />
             </geometry>
             <material name="gray"/>
@@ -137,7 +136,7 @@
         </collision>
         <visual>
-            <origin xyz="-${wheel_radius} ${wheel_radius} -${wheel_length/2}" rpy="${pi/2} 0 0"/>
+            <origin xyz="0 0 ${wheel_length/2}" rpy="-${pi/2} 0 0"/>
             <geometry>
-                <mesh filename="${wheel_mesh_file}" scale="${wheel_mesh_scale}" />
+                <mesh filename="${wheel_mesh_file}" scale="${mesh_scale}" />
             </geometry>
             <material name="gray"/>

Commit message: description/robot24_core.xacro: Add 3D camera to front of robot chassis
- Most likley will be relocated later

File: description/robot24_core.xacro (robot description, xacro)
@@ -146,3 +146,23 @@
         </xacro:inertial_cylinder>
     </link>
+    <!-- 3D Camera -->
+    <joint name="depth_camera_joint" type="fixed">
+        <parent link="chassis"/>
+        <child link="depth_camera"/>
+        <origin xyz="${chassis_length/2 + 0.0254} 0 0" rpy="0 0 0"/>
+    </joint>
+    <link name="depth_camera">
+        <visual>
+            <geometry>
+                <box size="0.010 0.03 0.03"/>
+            </geometry>
+            <material name="black"/>
+        </visual>
+        <visual>
+            <origin xyz="0 0 0"/>
+            <geometry>
+                <cylinder radius="0.002" length="0.1"/>
+            </geometry>
+        </visual>
+    </link>
 </robot>

Commit message: description/robot24_core.xacro: Added lidar floating at ~2ft height

File: description/robot24_core.xacro (robot description, xacro)
@@ -7,4 +7,7 @@
     <xacro:property name="chassis_height" value="0.0889" />
     <xacro:property name="chassis_width" value="0.3556" />
+    <xacro:property name="lidar_length" value="0.12954" />
+    <xacro:property name="lidar_height" value="0.07874" />
+    <xacro:property name="lidar_width" value="0.09906" />
     <xacro:property name="mesh_scale" value="0.001 0.001 0.001" />
     <xacro:property name="wheel_gap" value="0.0127" />
@@ -146,4 +149,28 @@
         </xacro:inertial_cylinder>
     </link>
+    <!-- 360 Lidar -->
+    <joint name="lidar_joint" type="fixed">
+        <parent link="chassis"/>
+        <child link="lidar"/>
+        <axis xyz="0 0 1"/>
+        <origin xyz="-${chassis_length/2} 0 0.6096" rpy="0 0 0"/>
+    </joint>
+    <link name="lidar">
+        <collision>
+            <geometry>
+                <box size="${lidar_length} ${lidar_width} ${lidar_height}"/>
+            </geometry>
+        </collision>
+        <visual>
+            <origin xyz="0 0 0" rpy="0 0 0"/>
+            <geometry>
+                <mesh filename="file://$(find osprey_ros)/meshes/rplidar.dae" scale="1 1 1" />
+            </geometry>
+            <material name="gray"/>
+        </visual>
+        <xacro:inertial_box mass="0.0001" x="${lidar_length}" y="${lidar_width}" z="0.6096">
+            <origin xyz="${lidar_length/2} ${lidar_width/2} 0.6096" rpy="0 0 0"/>
+        </xacro:inertial_box>
+    </link>
     <!-- 3D Camera -->
     <joint name="depth_camera_joint" type="fixed">

Commit message: description/robot24_core.xacro: Change lidar color to black from gray

File: description/robot24_core.xacro (robot description, xacro)
@@ -167,5 +167,5 @@
                 <mesh filename="file://$(find osprey_ros)/meshes/rplidar.dae" scale="1 1 1" />
             </geometry>
-            <material name="gray"/>
+            <material name="black"/>
         </visual>
         <xacro:inertial_box mass="0.0001" x="${lidar_length}" y="${lidar_width}" z="0.6096">

Commit message: description/robot24_core.xacro: Added excavation/deposition frame to model

File: description/robot24_core.xacro (robot description, xacro)
@@ -4,4 +4,8 @@
     <xacro:property name="limit_effort" value="100" />
     <xacro:property name="limit_velocity" value="10" />
+    <xacro:property name="bucket_frame_length" value="0.0508" /> <!-- depth -->
+    <xacro:property name="bucket_frame_height" value="0.4064" />
+    <xacro:property name="bucket_frame_width" value="${chassis_width}" />
+    <xacro:property name="bucket_frame_offset" value="${chassis_length/2 + buckets_width/10}" />
     <xacro:property name="chassis_length" value="0.8128" />
     <xacro:property name="chassis_height" value="0.0889" />
@@ -149,4 +153,29 @@
         </xacro:inertial_cylinder>
     </link>
+    <!-- Bucket Frame -->
+    <joint name="bucket_frame_joint" type="fixed">
+        <parent link="chassis"/>
+        <child link="bucket_frame"/>
+        <origin xyz="${chassis_length/4 + 0.0381} -0.00635 ${wheel_radius + 0.0277}" rpy="0 0 0"/>
+    </joint>
+    <link name="bucket_frame">
+        <collision>
+            <origin xyz="0 0 0" rpy="0 0 0"/>
+            <geometry>
+                <box size="${bucket_frame_length * collision_multiplier} ${bucket_frame_width * collision_multiplier} ${bucket_frame_height}"/>
+            </geometry>
+            <material name="gray"/>
+        </collision>
+        <visual>
+            <origin xyz="0 0 0" rpy="0 0 0"/>
+            <geometry>
+                <mesh filename="file://$(find osprey_ros)/meshes/robot24/exc_dep_frame.dae" scale="${mesh_scale}" />
+            </geometry>
+            <material name="gray"/>
+        </visual>
+        <xacro:inertial_box mass="0.05" x="${bucket_frame_length}" y="${bucket_frame_width}" z="${bucket_frame_height}">
+            <origin xyz="0 0 ${bucket_frame_height/2}" rpy="0 0 0"/>
+        </xacro:inertial_box>
+    </link>
     <!-- 360 Lidar -->
     <joint name="lidar_joint" type="fixed">

Commit message: description/robot24_core.xacro: Increase wheel radius to 5.6"/0.14224M

File: description/robot24_core.xacro (robot description, xacro)
@@ -17,5 +17,5 @@
     <xacro:property name="wheel_gap" value="0.0127" />
     <xacro:property name="wheel_length" value="0.1016" />
-    <xacro:property name="wheel_radius" value="0.1397" />
+    <xacro:property name="wheel_radius" value="0.14224" />
     <xacro:property name="wheel_mass" value="0.0624" />
     <xacro:property name="wheel_mesh_file" value="file://$(find osprey_ros)/meshes/robot24/wheel.dae" />

Commit message: description/robot24_core.xacro: Remove default 0 0 0 origin

File: description/robot24_core.xacro (robot description, xacro)
@@ -161,5 +161,4 @@
     <link name="bucket_frame">
         <collision>
-            <origin xyz="0 0 0" rpy="0 0 0"/>
             <geometry>
                 <box size="${bucket_frame_length * collision_multiplier} ${bucket_frame_width * collision_multiplier} ${bucket_frame_height}"/>
@@ -168,5 +167,4 @@
         </collision>
         <visual>
-            <origin xyz="0 0 0" rpy="0 0 0"/>
             <geometry>
                 <mesh filename="file://$(find osprey_ros)/meshes/robot24/exc_dep_frame.dae" scale="${mesh_scale}" />
@@ -192,5 +190,4 @@
         </collision>
         <visual>
-            <origin xyz="0 0 0" rpy="0 0 0"/>
             <geometry>
                 <mesh filename="file://$(find osprey_ros)/meshes/rplidar.dae" scale="1 1 1" />

Commit message: description/robot24_core.xacro: Added dig/dump bucket to model temp type
- The joint is temporarily added as prismatic but will most likely be
  switched over to floating

File: description/robot24_core.xacro (robot description, xacro)
@@ -4,4 +4,7 @@
     <xacro:property name="limit_effort" value="100" />
     <xacro:property name="limit_velocity" value="10" />
+    <xacro:property name="bucket_length" value="0.3556" /> <!-- depth -->
+    <xacro:property name="bucket_height" value="0.254" />
+    <xacro:property name="bucket_width" value="0.254" />
     <xacro:property name="bucket_frame_length" value="0.0508" /> <!-- depth -->
     <xacro:property name="bucket_frame_height" value="0.4064" />
@@ -176,4 +179,28 @@
         </xacro:inertial_box>
     </link>
+    <!-- Dig/Dump Bucket -->
+    <joint name="bucket_joint" type="prismatic">
+        <parent link="bucket_frame"/>
+        <child link="bucket"/>
+        <limit lower="-1"  upper="2"  velocity="0.1"  effort="${limit_effort}"  />
+        <axis xyz="0 0 1"/>
+        <origin xyz="-${bucket_length/2 + bucket_frame_length/2} 0 -${bucket_height/2}" rpy="0 0 0"/>
+    </joint>
+    <link name="bucket">
+        <collision>
+            <geometry>
+                <box size="${bucket_length} ${bucket_width} ${bucket_height}"/>
+            </geometry>
+        </collision>
+        <visual>
+            <geometry>
+                <mesh filename="file://$(find osprey_ros)/meshes/robot24/bucket.dae" scale="${mesh_scale}" />
+            </geometry>
+            <material name="gray"/>
+        </visual>
+        <xacro:inertial_box mass="0.1" x="${bucket_length}" y="${bucket_width}" z="${bucket_height}">
+            <origin xyz="${chassis_length/2} 0 ${bucket_height/2}" rpy="0 0 0"/>
+        </xacro:inertial_box>
+    </link>
     <!-- 360 Lidar -->
     <joint name="lidar_joint" type="fixed">

Commit message: description/robot24_core.xacro: Increase bucket frame depth/length

File: description/robot24_core.xacro (robot description, xacro)
@@ -7,5 +7,5 @@
     <xacro:property name="bucket_height" value="0.254" />
     <xacro:property name="bucket_width" value="0.254" />
-    <xacro:property name="bucket_frame_length" value="0.0508" /> <!-- depth -->
+    <xacro:property name="bucket_frame_length" value="0.1524" /> <!-- depth -->
     <xacro:property name="bucket_frame_height" value="0.4064" />
     <xacro:property name="bucket_frame_width" value="${chassis_width}" />

Commit message: description/robot24_core.xacro: Lower lidar to 18" above frame from 24"

File: description/robot24_core.xacro (robot description, xacro)
@@ -208,5 +208,5 @@
         <child link="lidar"/>
         <axis xyz="0 0 1"/>
-        <origin xyz="-${chassis_length/2} 0 0.6096" rpy="0 0 0"/>
+        <origin xyz="-${chassis_length/2} 0 0.4572" rpy="0 0 0"/>
     </joint>
     <link name="lidar">

Commit message: description/robot24_core.xacro: Corrected dimensions and alignment
- Corrected chassis dimensions to match the new robot
- Adjust wheel offsets and split up right/left offset variables/values

File: description/robot24_core.xacro (robot description, xacro)
@@ -11,7 +11,7 @@
     <xacro:property name="bucket_frame_width" value="${chassis_width}" />
     <xacro:property name="bucket_frame_offset" value="${chassis_length/2 + buckets_width/10}" />
-    <xacro:property name="chassis_length" value="0.8128" />
-    <xacro:property name="chassis_height" value="0.0889" />
-    <xacro:property name="chassis_width" value="0.3556" />
+    <xacro:property name="chassis_length" value="0.8382" />
+    <xacro:property name="chassis_height" value="0.0508" />
+    <xacro:property name="chassis_width" value="0.4318" />
     <xacro:property name="lidar_length" value="0.12954" />
     <xacro:property name="lidar_height" value="0.07874" />
@@ -25,5 +25,6 @@
     <xacro:property name="wheel_offset_front" value="${chassis_length/2 - 0.1024}" />
     <xacro:property name="wheel_offset_rear" value="${-chassis_length/2 + 0.1024}" />
-    <xacro:property name="wheel_offset_side" value="${wheel_length/2 + chassis_width/2 + wheel_gap}" />
+    <xacro:property name="wheel_offset_left" value="${wheel_length/2 + chassis_width/2 + wheel_gap}" />
+    <xacro:property name="wheel_offset_right" value="-${wheel_length/2 + chassis_width/2 + wheel_gap*2}" />
     <link name="base_link"></link>
     <joint name="base_footprint_joint" type="fixed">
@@ -60,5 +61,5 @@
         <parent link="chassis"/>
         <child link="front_left_wheel"/>
-        <origin xyz="${wheel_offset_front} ${wheel_offset_side} 0" rpy="-${pi/2} 0 0"/>
+        <origin xyz="${wheel_offset_front} ${wheel_offset_left} 0" rpy="-${pi/2} 0 0"/>
         <axis xyz="0 0 1"/>
         <limit effort="${limit_effort}" velocity="${limit_velocity}"/>
@@ -71,5 +72,5 @@
         </collision>
         <visual>
-            <origin xyz="0 0 ${wheel_length/2}" rpy="-${pi/2} 0 0"/>
+            <origin xyz="0 0 0" rpy="-${pi/2} 0 0"/>
             <geometry>
                 <mesh filename="${wheel_mesh_file}" scale="${mesh_scale}" />
@@ -85,5 +86,5 @@
         <parent link="chassis"/>
         <child link="front_right_wheel"/>
-        <origin xyz="${wheel_offset_front} -${wheel_offset_side} 0" rpy="${pi/2} 0 0"/>
+        <origin xyz="${wheel_offset_front} ${wheel_offset_right} 0" rpy="${pi/2} 0 0"/>
         <axis xyz="0 0 -1"/>
         <limit effort="${limit_effort}" velocity="${limit_velocity}"/>
@@ -96,5 +97,5 @@
         </collision>
         <visual>
-            <origin xyz="0 0 ${wheel_length/2}" rpy="-${pi/2} 0 0"/>
+            <origin xyz="0 0 0" rpy="-${pi/2} 0 0"/>
             <geometry>
                 <mesh filename="${wheel_mesh_file}" scale="${mesh_scale}" />
@@ -110,5 +111,5 @@
         <parent link="chassis"/>
         <child link="rear_left_wheel"/>
-        <origin xyz="${wheel_offset_rear} ${wheel_offset_side} 0" rpy="-${pi/2} 0 0"/>
+        <origin xyz="${wheel_offset_rear} ${wheel_offset_left} 0" rpy="-${pi/2} 0 0"/>
         <axis xyz="0 0 1"/>
         <limit effort="${limit_effort}" velocity="${limit_velocity}"/>
@@ -121,5 +122,5 @@
         </collision>
         <visual>
-            <origin xyz="0 0 ${wheel_length/2}" rpy="-${pi/2} 0 0"/>
+            <origin xyz="0 0 0" rpy="-${pi/2} 0 0"/>
             <geometry>
                 <mesh filename="${wheel_mesh_file}" scale="${mesh_scale}" />
@@ -135,5 +136,5 @@
         <parent link="chassis"/>
         <child link="rear_right_wheel"/>
-        <origin xyz="${wheel_offset_rear} -${wheel_offset_side} 0" rpy="${pi/2} 0 0"/>
+        <origin xyz="${wheel_offset_rear} ${wheel_offset_right} 0" rpy="${pi/2} 0 0"/>
         <axis xyz="0 0 -1"/>
         <limit effort="${limit_effort}" velocity="${limit_velocity}"/>
@@ -146,5 +147,5 @@
         </collision>
         <visual>
-            <origin xyz="0 0 ${wheel_length/2}" rpy="-${pi/2} 0 0"/>
+            <origin xyz="0 0 0" rpy="-${pi/2} 0 0"/>
             <geometry>
                 <mesh filename="${wheel_mesh_file}" scale="${mesh_scale}" />

Commit message: description/robot24_core.xacro: Add theoretical electrical box to rear
- Theoretical electrical box dimensions 17"w x 12"h x 3"d/l

File: description/robot24_core.xacro (robot description, xacro)
@@ -4,4 +4,7 @@
     <xacro:property name="limit_effort" value="100" />
     <xacro:property name="limit_velocity" value="10" />
+    <xacro:property name="electrical_length" value="0.0762" /> <!-- depth -->
+    <xacro:property name="electrical_height" value="0.3048" />
+    <xacro:property name="electrical_width" value="${chassis_width}" />
     <xacro:property name="bucket_length" value="0.3556" /> <!-- depth -->
     <xacro:property name="bucket_height" value="0.254" />
@@ -204,4 +207,27 @@
         </xacro:inertial_box>
     </link>
+    <!-- Electrical Box -->
+    <joint name="electrical_joint" type="fixed">
+        <parent link="chassis"/>
+        <child link="electrical"/>
+        <origin xyz="-${chassis_length/2 - electrical_length/1.95} -0.006 ${wheel_radius + chassis_height/1.4}" rpy="0 0 0"/>
+    </joint>
+    <link name="electrical">
+        <collision>
+            <geometry>
+                <box size="${electrical_length * collision_multiplier} ${electrical_width * collision_multiplier} ${electrical_height}"/>
+            </geometry>
+            <material name="white"/>
+        </collision>
+        <visual>
+            <geometry>
+                <box size="${electrical_length} ${electrical_width} ${electrical_height}"/>
+            </geometry>
+            <material name="white"/>
+        </visual>
+        <xacro:inertial_box mass="0.1" x="${electrical_length}" y="${electrical_width}" z="${electrical_height}">
+            <origin xyz="0 0 ${electrical_height/2}" rpy="0 0 0"/>
+        </xacro:inertial_box>
+    </link>
     <!-- 360 Lidar -->
     <joint name="lidar_joint" type="fixed">

Commit message: description/robot24_core.xacro: Add theoretical electronics box to front
- Theoretical electronics box dimensions 17"w x 8"h x 4"d/l

File: description/robot24_core.xacro (robot description, xacro)
@@ -7,4 +7,7 @@
     <xacro:property name="electrical_height" value="0.3048" />
     <xacro:property name="electrical_width" value="${chassis_width}" />
+    <xacro:property name="electronics_length" value="0.1016" /> <!-- depth -->
+    <xacro:property name="electronics_height" value="0.2032" />
+    <xacro:property name="electronics_width" value="${chassis_width}" />
     <xacro:property name="bucket_length" value="0.3556" /> <!-- depth -->
     <xacro:property name="bucket_height" value="0.254" />
@@ -207,4 +210,27 @@
         </xacro:inertial_box>
     </link>
+    <!-- Electronics Box -->
+    <joint name="electronics_joint" type="fixed">
+        <parent link="chassis"/>
+        <child link="electronics"/>
+        <origin xyz="${chassis_length/2 - electronics_length/2} -0.006 ${wheel_radius - chassis_height/3.5}" rpy="0 0 0"/>
+    </joint>
+    <link name="electronics">
+        <collision>
+            <geometry>
+                <box size="${electronics_length * collision_multiplier} ${electronics_width * collision_multiplier} ${electronics_height}"/>
+            </geometry>
+            <material name="white"/>
+        </collision>
+        <visual>
+            <geometry>
+                <box size="${electronics_length} ${electronics_width} ${electronics_height}"/>
+            </geometry>
+            <material name="white"/>
+        </visual>
+        <xacro:inertial_box mass="0.1" x="${electronics_length}" y="${electronics_width}" z="${electronics_height}">
+            <origin xyz="0 0 ${electronics_height/2}" rpy="0 0 0"/>
+        </xacro:inertial_box>
+    </link>
     <!-- Electrical Box -->
     <joint name="electrical_joint" type="fixed">

Commit message: description/robot24_core.xacro: Remove the prototype front electrical box

File: description/robot24_core.xacro (robot description, xacro)
@@ -7,7 +7,4 @@
     <xacro:property name="electrical_height" value="0.3048" />
     <xacro:property name="electrical_width" value="${chassis_width}" />
-    <xacro:property name="electronics_length" value="0.1016" /> <!-- depth -->
-    <xacro:property name="electronics_height" value="0.2032" />
-    <xacro:property name="electronics_width" value="${chassis_width}" />
     <xacro:property name="bucket_length" value="0.3556" /> <!-- depth -->
     <xacro:property name="bucket_height" value="0.254" />
@@ -210,27 +207,4 @@
         </xacro:inertial_box>
     </link>
-    <!-- Electronics Box -->
-    <joint name="electronics_joint" type="fixed">
-        <parent link="chassis"/>
-        <child link="electronics"/>
-        <origin xyz="${chassis_length/2 - electronics_length/2} -0.006 ${wheel_radius - chassis_height/3.5}" rpy="0 0 0"/>
-    </joint>
-    <link name="electronics">
-        <collision>
-            <geometry>
-                <box size="${electronics_length * collision_multiplier} ${electronics_width * collision_multiplier} ${electronics_height}"/>
-            </geometry>
-            <material name="white"/>
-        </collision>
-        <visual>
-            <geometry>
-                <box size="${electronics_length} ${electronics_width} ${electronics_height}"/>
-            </geometry>
-            <material name="white"/>
-        </visual>
-        <xacro:inertial_box mass="0.1" x="${electronics_length}" y="${electronics_width}" z="${electronics_height}">
-            <origin xyz="0 0 ${electronics_height/2}" rpy="0 0 0"/>
-        </xacro:inertial_box>
-    </link>
     <!-- Electrical Box -->
     <joint name="electrical_joint" type="fixed">
