Commit message: description/robot24_core.xacro: Updated bucket mass, added variable

File: description/robot24_core.xacro (robot description, xacro)
@@ -10,4 +10,5 @@
     <xacro:property name="bucket_height" value="0.254" />
     <xacro:property name="bucket_width" value="0.254" />
+    <xacro:property name="bucket_mass" value="1.68" />
     <xacro:property name="bucket_frame_length" value="0.1524" /> <!-- depth -->
     <xacro:property name="bucket_frame_height" value="0.4064" />
@@ -203,5 +204,5 @@
             <material name="gray"/>
         </visual>
-        <xacro:inertial_box mass="0.1" x="${bucket_length}" y="${bucket_width}" z="${bucket_height}">
+        <xacro:inertial_box mass="${bucket_mass}" x="${bucket_length}" y="${bucket_width}" z="${bucket_height}">
             <origin xyz="${chassis_length/2} 0 ${bucket_height/2}" rpy="0 0 0"/>
         </xacro:inertial_box>

Commit message: description/robot24_core.xacro: Updated wheel mass

File: description/robot24_core.xacro (robot description, xacro)
@@ -25,5 +25,5 @@
     <xacro:property name="wheel_length" value="0.1016" />
     <xacro:property name="wheel_radius" value="0.14224" />
-    <xacro:property name="wheel_mass" value="0.0624" />
+    <xacro:property name="wheel_mass" value="1.451" />
     <xacro:property name="wheel_mesh_file" value="file://$(find osprey_ros)/meshes/robot24/wheel.dae" />
     <xacro:property name="wheel_offset_front" value="${chassis_length/2 - 0.1024}" />

Commit message: description/robot24_core.xacro: Updated chassic mass, added variable

File: description/robot24_core.xacro (robot description, xacro)
@@ -18,4 +18,5 @@
     <xacro:property name="chassis_height" value="0.0508" />
     <xacro:property name="chassis_width" value="0.4318" />
+    <xacro:property name="chassis_mass" value="7.8" /> <!-- with motors -->
     <xacro:property name="lidar_length" value="0.12954" />
     <xacro:property name="lidar_height" value="0.07874" />
@@ -57,5 +58,5 @@
             <material name="gray"/>
         </visual>
-        <xacro:inertial_box mass="2.5" x="${chassis_length}" y="${chassis_width}" z="${chassis_height}">
+        <xacro:inertial_box mass="${chassis_mass}" x="${chassis_length}" y="${chassis_width}" z="${chassis_height}">
             <origin xyz="0 0 0" rpy="0 0 0"/>
         </xacro:inertial_box>

Commit message: description/robot24_core.xacro: Update electrical box length and height

File: description/robot24_core.xacro (robot description, xacro)
@@ -4,6 +4,6 @@
     <xacro:property name="limit_effort" value="100" />
     <xacro:property name="limit_velocity" value="10" />
-    <xacro:property name="electrical_length" value="0.0762" /> <!-- depth -->
-    <xacro:property name="electrical_height" value="0.3048" />
+    <xacro:property name="electrical_length" value="0.2159" /> <!-- depth -->
+    <xacro:property name="electrical_height" value="0.2159" />
     <xacro:property name="electrical_width" value="${chassis_width}" />
     <xacro:property name="bucket_length" value="0.3556" /> <!-- depth -->
